Commit message: Fix base_footprint link, add rviz config, update launch with rviz path

File: final_robot_description/urdf/arm.xacro (robot description, xacro)
@@ -41,4 +41,5 @@
     </visual>
   </link>
+  <link name="base_footprint"/>
     <joint name="arm_base_joint" type="fixed">
       <parent link="base_footprint"/>
@@ -55,9 +56,10 @@
     </joint>
     <joint name="forearm_to_hand" type="revolute">
-      <parent link="forerm_link"/>
+      <parent link="forearm_link"/>
       <child link="hand_link"/>
-      <origin xyz="0 0 ${arm_base_height}" rpy="0 0 0"/>
+      <origin xyz="0 0 ${forearm_length}" rpy="0 0 0"/>
       <axis xyz="0 1 0"/>
       <limit lower="0" upper="${pi/2}" effort="100" velocity="100"/>
       <dynamics friction="0.05" damping="0.1"/>
     </joint>
+    </robot>

File: final_robot_description/urdf/standalone_arm.urdf.xacro (robot description, xacro)
@@ -1,2 +1,5 @@
+<?xml version="1.0"?>
+<robot name="standalone_arm" xmlns:xacro="http://www.ros.org/wiki/xacro">
 <xacro:include filename="$(find final_robot_description)/urdf/common_properties.xacro"/>
 <xacro:include filename="$(find final_robot_description)/urdf/arm.xacro"/>
+</robot>

Commit message: Add collision and inertial to arm.xacro

File: final_robot_description/urdf/arm.xacro (robot description, xacro)
@@ -18,4 +18,11 @@
       </material>
     </visual>
+    <collision>
+      <geometry>
+      <box size="${arm_base_length} ${arm_base_width} ${arm_base_height}"/>
+      </geometry>
+      <origin xyz="0 0 ${arm_base_height/2}" rpy="0 0 0"/>
+   </collision>
+   <xacro:inertial_box mass="5.0" x="${arm_base_length}" y="${arm_base_width}" z="${arm_base_height}"/>
   </link>
   <link name="forearm_link">
@@ -29,4 +36,11 @@
       </material>
     </visual>
+    <collision>
+      <geometry>
+      <cylinder radius="${forearm_radius}" length="${forearm_length}"/>
+      </geometry>
+      <origin xyz="0 0 ${forearm_length/2}" rpy="0 0 0"/>
+    </collision>
+    <xacro:inertial_cylinder mass="0.3" radius="${forearm_radius}" length="${forearm_length}"/>
   </link>
    <link name="hand_link">
@@ -40,4 +54,11 @@
       </material>
     </visual>
+    <collision>
+      <geometry>
+       <cylinder radius="${hand_radius}" length="${hand_length}"/>
+      </geometry>
+      <origin xyz="0 0 ${hand_length/2}" rpy="0 0 0"/>
+    </collision>
+    <xacro:inertial_cylinder mass="0.3" radius="${hand_radius}" length="${hand_length}"/>
   </link>
   <link name="base_footprint"/>

Commit message: Add collision, inertial, Gazebo material, Gazebo launch - Ders 58 complete

File: final_robot_description/urdf/arm.xacro (robot description, xacro)
@@ -23,6 +23,9 @@
       </geometry>
       <origin xyz="0 0 ${arm_base_height/2}" rpy="0 0 0"/>
-   </collision>
-   <xacro:inertial_box mass="5.0" x="${arm_base_length}" y="${arm_base_width}" z="${arm_base_height}"/>
+    </collision>
+    <xacro:inertial_box mass="5.0" x="${arm_base_length}" y="${arm_base_width}" z="${arm_base_height}"/>
+    <gazebo reference="arm_base_link">
+      <material>Gazebo/Orange</material>
+    </gazebo>
   </link>
   <link name="forearm_link">
@@ -43,4 +46,7 @@
     </collision>
     <xacro:inertial_cylinder mass="0.3" radius="${forearm_radius}" length="${forearm_length}"/>
+    <gazebo reference="forearm_link">
+      <material>Gazebo/Blue</material>
+    </gazebo>
   </link>
    <link name="hand_link">
@@ -61,4 +67,7 @@
     </collision>
     <xacro:inertial_cylinder mass="0.3" radius="${hand_radius}" length="${hand_length}"/>
+    <gazebo reference="hand_link">
+      <material>Gazebo/Orange</material>
+    </gazebo>
   </link>
   <link name="base_footprint"/>

Commit message: Add JointStatePublisher and JointPositionController plugins

File: final_robot_description/urdf/arm.xacro (robot description, xacro)
@@ -25,8 +25,8 @@
     </collision>
     <xacro:inertial_box mass="5.0" x="${arm_base_length}" y="${arm_base_width}" z="${arm_base_height}"/>
+  </link>
     <gazebo reference="arm_base_link">
       <material>Gazebo/Orange</material>
     </gazebo>
-  </link>
   <link name="forearm_link">
     <visual>
@@ -93,3 +93,24 @@
       <dynamics friction="0.05" damping="0.1"/>
     </joint>
+    <gazebo>
+     <plugin filename="gz-sim-joint-state-publisher-system"
+        name="gz::sim::systems::JointStatePublisher">
+     <joint_name>arm_base_to_forearm</joint_name>
+     <joint_name>forearm_to_hand</joint_name>
+     </plugin>
+    </gazebo>
+    <gazebo>
+      <plugin filename="gz-sim-joint-position-controller-system"
+        name="gz::sim::systems::JointPositionController">
+       <joint_name>arm_base_to_forearm</joint_name>
+       <p_gain>5.0</p_gain>
+      </plugin>
+    </gazebo>
+    <gazebo>
+      <plugin filename="gz-sim-joint-position-controller-system"
+         name="gz::sim::systems::JointPositionController">
+       <joint_name>forearm_to_hand</joint_name>
+       <p_gain>3.0</p_gain>
+      </plugin>
+    </gazebo>
     </robot>

Commit message: Combine arm and mobile base - Ders 60 complete

File: final_robot_description/urdf/arm.xacro (robot description, xacro)
@@ -24,5 +24,5 @@
       <origin xyz="0 0 ${arm_base_height/2}" rpy="0 0 0"/>
     </collision>
-    <xacro:inertial_box mass="5.0" x="${arm_base_length}" y="${arm_base_width}" z="${arm_base_height}"/>
+    <xacro:inertial_box mass="0.5" x="${arm_base_length}" y="${arm_base_width}" z="${arm_base_height}"/>
   </link>
     <gazebo reference="arm_base_link">
@@ -71,10 +71,4 @@
     </gazebo>
   </link>
-  <link name="base_footprint"/>
-    <joint name="arm_base_joint" type="fixed">
-      <parent link="base_footprint"/>
-      <child link="arm_base_link"/>
-      <origin xyz="0 0 ${arm_base_height/2}" rpy="0 0 0"/>
-    </joint>
     <joint name="arm_base_to_forearm" type="revolute">
       <parent link="arm_base_link"/>

File: final_robot_description/urdf/final_robot_full.urdf.xacro (robot description, xacro)
@@ -3,3 +3,9 @@
   <xacro:include filename="$(find final_robot_description)/urdf/common_properties.xacro"/>
   <xacro:include filename="$(find final_robot_description)/urdf/mobile_base.xacro"/>
+  <xacro:include filename="$(find final_robot_description)/urdf/arm.xacro"/>
+  <joint name="arm_base_joint" type="fixed">
+  <parent link="base_link"/>
+  <child link="arm_base_link"/>
+  <origin xyz="0 0 ${base_height}" rpy="0 0 0"/>
+</joint>
 </robot>
