Commit message: Combine arm and mobile base - Ders 60 complete

File: final_robot_description/urdf/final_robot_full.urdf.xacro (robot description, xacro)
@@ -7,5 +7,5 @@
   <parent link="base_link"/>
   <child link="arm_base_link"/>
-  <origin xyz="0 0 ${base_height}" rpy="0 0 0"/>
+  <origin xyz="${base_length/4} 0 ${base_height}" rpy="0 0 0"/>
 </joint>
 </robot>

File: final_robot_description/urdf/mobile_base.xacro (robot description, xacro)
@@ -32,5 +32,5 @@
       <origin xyz="0 0 ${base_height/2}" rpy="0 0 0"/>
     </collision>
-    <xacro:inertial_box mass="1.0" x="${base_length}" y="${base_width}" z="${base_height}"/>
+    <xacro:inertial_box mass="5.0" x="${base_length}" y="${base_width}" z="${base_height}"/>
   </link>
   <gazebo reference="base_link">
@@ -109,5 +109,5 @@
     <parent link="base_link"/>
     <child link="caster_wheel_link"/>
-    <origin xyz="${-base_length/2+caster_wheel_radius} 0 ${-(base_height/2-caster_wheel_radius)}" rpy="0 0 0"/>
+    <origin xyz="${base_length/2-caster_wheel_radius} 0 ${-(base_height/2-caster_wheel_radius)}" rpy="0 0 0"/>
   </joint>
   <gazebo reference="caster_wheel_link">
